File: drone_pdb.kicad_pcb (KiCad board)
At the start: 2 copper layers, 50.8 x 49.5 mm, 23 parts

Commit message: added pngs
Parts:
- moved Cin3 1.74 mm to (122.5, 72.5)
- moved Cin2 1.65 mm to (124.5, 72.7)
- moved Cin1 1.52 mm to (126.8, 72.7)
Routing:
- net VCC: track 1.54 -> 8.08 mm
